File: eagle/cell.sch (EAGLE design)
At the start: 11 parts

Commit message: add pcb text
Other:
- note added: "Harold Cooper"
- note added: "v0.1"
Changed lines of the file:
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@@
 <sheet>
 <plain>
+<text x="167.64" y="10.16" size="2.54" layer="94">Harold Cooper</text>
+<text x="238.76" y="7.62" size="2.54" layer="94">v0.1</text>
 </plain>
 <instances>

Commit message: cell v0.1, as ordered from OSH Park on 2014-10-07
Parts:
- removed U$1: XBEE-1XBEE-1_LOCK, SparkFun-RF:XBEE-1XBEE-1_LOCK
- added XB24: XBEE-1XBEE-1_LOCK, hrldcpr:XBEE-1XBEE-1_LOCK
- MCP1700: value (none) -> MCP1700; device adafruit:MCP1700INLINE -> hrldcpr:MCP1700
- MCP9700A: value MCP9700A-E/TO -> (none); device Microchip_By_element14_Batch_1:MCP9700A-E/TO -> SparkFun-Connectors:M03LOCK
Connections:
- net 3.3V: now also MCP1700.3.3V, XB24.VCC, XB24.VREF; no longer MCP1700.OUT, U$1.RES@14, U$1.VDD
- net GND: now also MCP9700A.3, XB24.GND; no longer MCP9700A.GND, U$1.GND
- net N$1: now also MCP9700A.1; no longer MCP9700A.VDD
- net N$2: now also XB24.ON; no longer U$1.DIO9
- net N$3: now also MCP9700A.2, XB24.DIO0; no longer MCP9700A.VOUT, U$1.DIO0
Changed lines of the file:
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@@
 <part name="GND3" library="SparkFun-Aesthetics" deviceset="GND" device=""/>
 <part name="SUPPLY4" library="SparkFun-Aesthetics" deviceset="3.3V" device=""/>
-<part name="MCP1700" library="adafruit" deviceset="MCP1700" device="INLINE"/>
-<part name="MCP9700A" library="Microchip_By_element14_Batch_1" deviceset="MCP9700A-E/TO" device=""/>
 <part name="C1" library="SparkFun-Capacitors" deviceset="CAP" device="0805" value="1µF"/>
-<part name="C2" library="SparkFun-Capacitors" deviceset="CAP" device="0805" value="1µF"/>
 <part name="C3" library="SparkFun-Capacitors" deviceset="CAP" device="0805" value="1µF"/>
 <part name="C4" library="SparkFun-Capacitors" deviceset="CAP" device="0805" value="8.2pF"/>
@@
 <part name="C6" library="SparkFun-Capacitors" deviceset="CAP" device="0805" value="1µF"/>
 <part name="R1" library="SparkFun-Resistors" deviceset="RESISTOR" device="0805-RES" value="200Ω"/>
-<part name="U$1" library="SparkFun-RF" deviceset="XBEE-1" device="XBEE-1_LOCK"/>
+<part name="XB24" library="hrldcpr" deviceset="XBEE-1" device="XBEE-1_LOCK"/>
+<part name="MCP1700" library="hrldcpr" deviceset="MCP1700" device=""/>
+<part name="C2" library="SparkFun-Capacitors" deviceset="CAP" device="0805" value="1µF"/>
+<part name="MCP9700A" library="SparkFun-Connectors" deviceset="M03" device="LOCK"/>
 </parts>
 <sheets>
@@
 <instance part="GND3" gate="1" x="137.16" y="71.12"/>
 <instance part="SUPPLY4" gate="G$1" x="127" y="83.82"/>
-<instance part="MCP1700" gate="1" x="104.14" y="119.38"/>
-<instance part="MCP9700A" gate="A" x="162.56" y="81.28"/>
 <instance part="C1" gate="G$1" x="88.9" y="114.3"/>
-<instance part="C2" gate="G$1" x="119.38" y="114.3"/>
 <instance part="C3" gate="G$1" x="68.58" y="93.98"/>
 <instance part="C4" gate="G$1" x="76.2" y="93.98"/>
@@
 <instance part="C6" gate="G$1" x="137.16" y="76.2"/>
 <instance part="R1" gate="G$1" x="132.08" y="81.28"/>
-<instance part="U$1" gate="G$1" x="104.14" y="88.9"/>
+<instance part="XB24" gate="G$1" x="104.14" y="88.9"/>
+<instance part="MCP1700" gate="G$1" x="104.14" y="119.38"/>
+<instance part="C2" gate="G$1" x="119.38" y="114.3"/>
+<instance part="MCP9700A" gate="G$1" x="154.94" y="78.74" rot="R180"/>
 </instances>
 <busses>
@@
 <segment>
 <pinref part="GND1" gate="1" pin="GND"/>
-<pinref part="MCP1700" gate="1" pin="GND"/>
 <pinref part="C1" gate="G$1" pin="2"/>
 <wire x1="88.9" y1="111.76" x2="104.14" y2="111.76" width="0.1524" layer="91"/>
 <junction x="104.14" y="111.76"/>
+<pinref part="MCP1700" gate="G$1" pin="GND"/>
 <pinref part="C2" gate="G$1" pin="2"/>
-<wire x1="104.14" y1="111.76" x2="119.38" y2="111.76" width="0.1524" layer="91"/>
+<wire x1="119.38" y1="111.76" x2="104.14" y2="111.76" width="0.1524" layer="91"/>
 </segment>
 <segment>
@@
 <pinref part="C6" gate="G$1" pin="2"/>
 <pinref part="C6" gate="G$1" pin="2"/>
-<pinref part="MCP9700A" gate="A" pin="GND"/>
 <wire x1="144.78" y1="76.2" x2="144.78" y2="73.66" width="0.1524" layer="91"/>
 <wire x1="144.78" y1="73.66" x2="137.16" y2="73.66" width="0.1524" layer="91"/>
 <junction x="137.16" y="73.66"/>
+<pinref part="MCP9700A" gate="G$1" pin="3"/>
+<wire x1="144.78" y1="76.2" x2="147.32" y2="76.2" width="0.1524" layer="91"/>
 </segment>
 <segment>
@@
 <wire x1="76.2" y1="91.44" x2="76.2" y2="76.2" width="0.1524" layer="91"/>
 <junction x="76.2" y="76.2"/>
-<pinref part="U$1" gate="G$1" pin="GND"/>
+<pinref part="XB24" gate="G$1" pin="GND"/>
 </segment>
 </net>
@@
 <wire x1="76.2" y1="99.06" x2="83.82" y2="99.06" width="0.1524" layer="91"/>
 <junction x="76.2" y="99.06"/>
-<pinref part="U$1" gate="G$1" pin="VDD"/>
+<pinref part="XB24" gate="G$1" pin="VCC"/>
+</segment>
+<segment>
+<pinref part="SUPPLY4" gate="G$1" pin="3.3V"/>
+<wire x1="127" y1="83.82" x2="124.46" y2="83.82" width="0.1524" layer="91"/>
+<pinref part="XB24" gate="G$1" pin="VREF"/>
 </segment>
 <segment>
 <pinref part="SUPPLY2" gate="G$1" pin="3.3V"/>
 <pinref part="C2" gate="G$1" pin="1"/>
-<pinref part="C2" gate="G$1" pin="1"/>
-<pinref part="MCP1700" gate="1" pin="OUT"/>
+<pinref part="MCP1700" gate="G$1" pin="3.3V"/>
 <wire x1="119.38" y1="119.38" x2="111.76" y2="119.38" width="0.1524" layer="91"/>
 <junction x="119.38" y="119.38"/>
-</segment>
-<segment>
-<pinref part="SUPPLY4" gate="G$1" pin="3.3V"/>
-<wire x1="127" y1="83.82" x2="124.46" y2="83.82" width="0.1524" layer="91"/>
-<pinref part="U$1" gate="G$1" pin="RES@14"/>
 </segment>
 </net>
@@
 <pinref part="C1" gate="G$1" pin="1"/>
 <pinref part="C1" gate="G$1" pin="1"/>
-<pinref part="MCP1700" gate="1" pin="IN"/>
 <wire x1="88.9" y1="119.38" x2="96.52" y2="119.38" width="0.1524" layer="91"/>
 <junction x="88.9" y="119.38"/>
+<pinref part="MCP1700" gate="G$1" pin="IN"/>
 </segment>
 </net>
@@
 <pinref part="C6" gate="G$1" pin="1"/>
 <pinref part="R1" gate="G$1" pin="2"/>
-<pinref part="MCP9700A" gate="A" pin="VDD"/>
-<wire x1="144.78" y1="81.28" x2="137.16" y2="81.28" width="0.1524" layer="91"/>
+<wire x1="147.32" y1="81.28" x2="137.16" y2="81.28" width="0.1524" layer="91"/>
 <junction x="137.16" y="81.28"/>
+<pinref part="MCP9700A" gate="G$1" pin="1"/>
 </segment>
 </net>
@@
 <pinref part="R1" gate="G$1" pin="1"/>
 <wire x1="124.46" y1="81.28" x2="127" y2="81.28" width="0.1524" layer="91"/>
-<pinref part="U$1" gate="G$1" pin="DIO9"/>
+<pinref part="XB24" gate="G$1" pin="ON"/>
 </segment>
 </net>
@@
 <pinref part="C5" gate="G$1" pin="1"/>
 <wire x1="137.16" y1="99.06" x2="124.46" y2="99.06" width="0.1524" layer="91"/>
-<pinref part="MCP9700A" gate="A" pin="VOUT"/>
-<wire x1="137.16" y1="99.06" x2="180.34" y2="99.06" width="0.1524" layer="91"/>
-<wire x1="180.34" y1="99.06" x2="180.34" y2="78.74" width="0.1524" layer="91"/>
+<wire x1="137.16" y1="99.06" x2="144.78" y2="99.06" width="0.1524" layer="91"/>
+<wire x1="144.78" y1="99.06" x2="144.78" y2="78.74" width="0.1524" layer="91"/>
 <junction x="137.16" y="99.06"/>
-<pinref part="U$1" gate="G$1" pin="DIO0"/>
+<pinref part="XB24" gate="G$1" pin="DIO0"/>
+<pinref part="MCP9700A" gate="G$1" pin="2"/>
+<wire x1="144.78" y1="78.74" x2="147.32" y2="78.74" width="0.1524" layer="91"/>
 </segment>
 </net>
