File: hub/hub.sch (EAGLE design)
At the start: 5 parts

Commit message: smd-ver
Parts:
- removed Rπ: M9X2, hrldcpr:M9X2
- removed XB24: XBEE-1XBEE-1, hrldcpr:XBEE-1XBEE-1
- added 3.3VPI: S5718-NDSMD, heatseek_hub_smd_lib:S5718-NDSMD
- added U$1: XBEESMD, heatseek_hub_smd_lib:XBEESMD
Connections:
- net 3.3V: now also 3.3VPI.1, 3.3VPI.17, U$1.1-VCC; no longer Rπ.1, Rπ.17, XB24.VCC
- net GND: now also 3.3VPI.14, 3.3VPI.6, 3.3VPI.9, U$1.10-GND; no longer Rπ.14, Rπ.6, Rπ.9, XB24.GND
- net N$1: now also 3.3VPI.10, U$1.2-DOUT; no longer Rπ.10, XB24.DOUT
- net N$2: now also 3.3VPI.8, U$1.3-DIN; no longer Rπ.8, XB24.DIN
Changed lines of the file:
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@@
 <?xml version="1.0" encoding="utf-8"?>
 <!DOCTYPE eagle SYSTEM "eagle.dtd">
-<eagle version="7.1.0">
+<eagle version="7.3.0">
 <drawing>
 <settings>
@@
 <layer number="56" name="wert" color="7" fill="1" visible="no" active="no"/>
 <layer number="57" name="tCAD" color="7" fill="1" visible="no" active="no"/>
+<layer number="59" name="tCarbon" color="7" fill="1" visible="no" active="no"/>
+<layer number="60" name="bCarbon" color="7" fill="1" visible="no" active="no"/>
 <layer number="90" name="Modules" color="5" fill="1" visible="yes" active="yes"/>
 <layer number="91" name="Nets" color="2" fill="1" visible="yes" active="yes"/>
@@
 <layer number="112" name="tSilk" color="7" fill="1" visible="yes" active="yes"/>
 <layer number="113" name="IDFDebug" color="4" fill="1" visible="yes" active="yes"/>
+<layer number="114" name="Badge_Outline" color="7" fill="1" visible="yes" active="yes"/>
+<layer number="115" name="ReferenceISLANDS" color="7" fill="1" visible="yes" active="yes"/>
 <layer number="116" name="Patch_BOT" color="9" fill="4" visible="yes" active="yes"/>
+<layer number="118" name="Rect_Pads" color="7" fill="1" visible="yes" active="yes"/>
 <layer number="121" name="_tsilk" color="7" fill="1" visible="yes" active="yes"/>
 <layer number="122" name="_bsilk" color="7" fill="1" visible="yes" active="yes"/>
@@
 <layer number="127" name="_tValues" color="7" fill="1" visible="yes" active="yes"/>
 <layer number="128" name="_bValues" color="7" fill="1" visible="yes" active="yes"/>
+<layer number="129" name="Mask" color="7" fill="1" visible="yes" active="yes"/>
 <layer number="131" name="tAdjust" color="7" fill="1" visible="yes" active="yes"/>
 <layer number="132" name="bAdjust" color="7" fill="1" visible="yes" active="yes"/>
@@
 <layer number="223" name="223bmp" color="24" fill="1" visible="no" active="no"/>
 <layer number="224" name="224bmp" color="25" fill="1" visible="no" active="no"/>
+<layer number="225" name="225bmp" color="7" fill="1" visible="yes" active="yes"/>
+<layer number="226" name="226bmp" color="7" fill="1" visible="yes" active="yes"/>
+<layer number="227" name="227bmp" color="7" fill="1" visible="yes" active="yes"/>
+<layer number="228" name="228bmp" color="7" fill="1" visible="yes" active="yes"/>
+<layer number="229" name="229bmp" color="7" fill="1" visible="yes" active="yes"/>
+<layer number="230" name="230bmp" color="7" fill="1" visible="yes" active="yes"/>
+<layer number="231" name="231bmp" color="7" fill="1" visible="yes" active="yes"/>
 <layer number="248" name="Housing" color="7" fill="1" visible="yes" active="yes"/>
 <layer number="249" name="Edge" color="7" fill="1" visible="yes" active="yes"/>
@@
 <layer number="251" name="SMDround" color="12" fill="11" visible="no" active="no"/>
 <layer number="254" name="cooling" color="7" fill="1" visible="yes" active="yes"/>
+<layer number="255" name="routoute" color="7" fill="1" visible="yes" active="yes"/>
 </layers>
 <schematic xreflabel="%F%N/%S.%C%R" xrefpart="/%S.%C%R">
@@
 </variantdefs>
 <classes>
-<class number="0" name="default" width="0" drill="0">
+<class number="0" name="default" width="0.4064" drill="0">
 </class>
 </classes>
 <parts>
 <part name="FRAME1" library="SparkFun-Aesthetics" deviceset="FRAME-LETTER" device=""/>
-<part name="XB24" library="hrldcpr" deviceset="XBEE-1" device="XBEE-1"/>
-<part name="Rπ" library="hrldcpr" deviceset="M9X2" device=""/>
 <part name="SUPPLY1" library="SparkFun-Aesthetics" deviceset="3.3V" device=""/>
 <part name="GND1" library="SparkFun-Aesthetics" deviceset="GND" device=""/>
@@
 <part name="GND3" library="SparkFun-Aesthetics" deviceset="GND" device=""/>
 <part name="SUPPLY2" library="SparkFun-Aesthetics" deviceset="3.3V" device=""/>
+<part name="U$1" library="heatseek_hub_smd_lib" deviceset="XBEE" device="SMD"/>
+<part name="3.3VPI" library="heatseek_hub_smd_lib" deviceset="S5718-ND" device="SMD"/>
 </parts>
 <sheets>
@@
 <instance part="FRAME1" gate="G$1" x="0" y="0"/>
 <instance part="FRAME1" gate="G$2" x="147.32" y="0"/>
-<instance part="XB24" gate="G$1" x="119.38" y="101.6"/>
-<instance part="Rπ" gate="G$1" x="63.5" y="111.76"/>
-<instance part="SUPPLY1" gate="G$1" x="55.88" y="121.92"/>
-<instance part="GND1" gate="1" x="53.34" y="109.22"/>
-<instance part="GND2" gate="1" x="78.74" y="114.3"/>
+<instance part="SUPPLY1" gate="G$1" x="20.32" y="127"/>
+<instance part="GND1" gate="1" x="17.78" y="104.14"/>
+<instance part="GND2" gate="1" x="53.34" y="114.3"/>
 <instance part="SUPPLY3" gate="G$1" x="83.82" y="111.76"/>
 <instance part="GND4" gate="1" x="83.82" y="86.36"/>
 <instance part="C1" gate="G$1" x="83.82" y="106.68"/>
 <instance part="C2" gate="G$1" x="91.44" y="106.68"/>
-<instance part="GND3" gate="1" x="73.66" y="104.14"/>
-<instance part="SUPPLY2" gate="G$1" x="50.8" y="101.6"/>
+<instance part="GND3" gate="1" x="53.34" y="93.98"/>
+<instance part="SUPPLY2" gate="G$1" x="17.78" y="86.36"/>
+<instance part="U$1" gate="G$1" x="119.38" y="101.6"/>
+<instance part="3.3VPI" gate="G$1" x="35.56" y="106.68"/>
 </instances>
 <busses>
@@
 <net name="3.3V" class="0">
 <segment>
-<pinref part="Rπ" gate="G$1" pin="1"/>
-<pinref part="SUPPLY1" gate="G$1" pin="3.3V"/>
-</segment>
-<segment>
 <pinref part="SUPPLY3" gate="G$1" pin="3.3V"/>
 <pinref part="C1" gate="G$1" pin="1"/>
@@
 <wire x1="83.82" y1="111.76" x2="91.44" y2="111.76" width="0.1524" layer="91"/>
 <junction x="83.82" y="111.76"/>
-<wire x1="91.44" y1="111.76" x2="99.06" y2="111.76" width="0.1524" layer="91"/>
+<wire x1="91.44" y1="111.76" x2="101.6" y2="111.76" width="0.1524" layer="91"/>
 <junction x="91.44" y="111.76"/>
-<pinref part="XB24" gate="G$1" pin="VCC"/>
-</segment>
-<segment>
-<pinref part="Rπ" gate="G$1" pin="17"/>
+<pinref part="U$1" gate="G$1" pin="1-VCC"/>
+</segment>
+<segment>
+<pinref part="SUPPLY1" gate="G$1" pin="3.3V"/>
+<pinref part="3.3VPI" gate="G$1" pin="1"/>
+<wire x1="20.32" y1="127" x2="22.86" y2="127" width="0.1524" layer="91"/>
+</segment>
+<segment>
 <pinref part="SUPPLY2" gate="G$1" pin="3.3V"/>
-<wire x1="50.8" y1="101.6" x2="55.88" y2="101.6" width="0.1524" layer="91"/>
+<pinref part="3.3VPI" gate="G$1" pin="17"/>
+<wire x1="17.78" y1="86.36" x2="22.86" y2="86.36" width="0.1524" layer="91"/>
 </segment>
 </net>
 <net name="GND" class="0">
-<segment>
-<pinref part="Rπ" gate="G$1" pin="9"/>
-<pinref part="GND1" gate="1" pin="GND"/>
-<wire x1="53.34" y1="111.76" x2="55.88" y2="111.76" width="0.1524" layer="91"/>
-</segment>
-<segment>
-<pinref part="Rπ" gate="G$1" pin="6"/>
-<pinref part="GND2" gate="1" pin="GND"/>
-<wire x1="71.12" y1="116.84" x2="78.74" y2="116.84" width="0.1524" layer="91"/>
-</segment>
 <segment>
 <pinref part="C1" gate="G$1" pin="2"/>
 <pinref part="GND4" gate="1" pin="GND"/>
 <wire x1="83.82" y1="104.14" x2="83.82" y2="88.9" width="0.1524" layer="91"/>
-<wire x1="99.06" y1="88.9" x2="91.44" y2="88.9" width="0.1524" layer="91"/>
+<wire x1="101.6" y1="88.9" x2="91.44" y2="88.9" width="0.1524" layer="91"/>
 <junction x="83.82" y="88.9"/>
 <pinref part="C2" gate="G$1" pin="2"/>
@@
 <wire x1="91.44" y1="104.14" x2="91.44" y2="88.9" width="0.1524" layer="91"/>
 <junction x="91.44" y="88.9"/>
-<pinref part="XB24" gate="G$1" pin="GND"/>
-</segment>
-<segment>
-<pinref part="Rπ" gate="G$1" pin="14"/>
+<pinref part="U$1" gate="G$1" pin="10-GND"/>
+</segment>
+<segment>
+<pinref part="GND1" gate="1" pin="GND"/>
+<pinref part="3.3VPI" gate="G$1" pin="9"/>
+<wire x1="17.78" y1="106.68" x2="22.86" y2="106.68" width="0.1524" layer="91"/>
+</segment>
+<segment>
+<pinref part="3.3VPI" gate="G$1" pin="14"/>
 <pinref part="GND3" gate="1" pin="GND"/>
-<wire x1="73.66" y1="106.68" x2="71.12" y2="106.68" width="0.1524" layer="91"/>
+<wire x1="48.26" y1="96.52" x2="53.34" y2="96.52" width="0.1524" layer="91"/>
+</segment>
+<segment>
+<pinref part="3.3VPI" gate="G$1" pin="6"/>
+<pinref part="GND2" gate="1" pin="GND"/>
+<wire x1="48.26" y1="116.84" x2="53.34" y2="116.84" width="0.1524" layer="91"/>
 </segment>
 </net>
 <net name="N$2" class="0">
 <segment>
-<pinref part="Rπ" gate="G$1" pin="8"/>
-<wire x1="71.12" y1="114.3" x2="76.2" y2="114.3" width="0.1524" layer="91"/>
-<wire x1="76.2" y1="114.3" x2="76.2" y2="106.68" width="0.1524" layer="91"/>
-<pinref part="XB24" gate="G$1" pin="DIN"/>
-<wire x1="76.2" y1="106.68" x2="99.06" y2="106.68" width="0.1524" layer="91"/>
+<wire x1="66.04" y1="106.68" x2="101.6" y2="106.68" width="0.1524" layer="91"/>
+<pinref part="U$1" gate="G$1" pin="3-DIN"/>
+<wire x1="66.04" y1="106.68" x2="66.04" y2="111.76" width="0.1524" layer="91"/>
+<pinref part="3.3VPI" gate="G$1" pin="8"/>
+<wire x1="66.04" y1="111.76" x2="48.26" y2="111.76" width="0.1524" layer="91"/>
 </segment>
 </net>
 <net name="N$1" class="0">
 <segment>
-<pinref part="XB24" gate="G$1" pin="DOUT"/>
-<wire x1="73.66" y1="109.22" x2="99.06" y2="109.22" width="0.1524" layer="91"/>
-<pinref part="Rπ" gate="G$1" pin="10"/>
-<wire x1="71.12" y1="111.76" x2="73.66" y2="111.76" width="0.1524" layer="91"/>
-<wire x1="73.66" y1="111.76" x2="73.66" y2="109.22" width="0.1524" layer="91"/>
-</segment>
-</net>
+<wire x1="53.34" y1="109.22" x2="101.6" y2="109.22" width="0.1524" layer="91"/>
+<pinref part="U$1" gate="G$1" pin="2-DOUT"/>
+<wire x1="53.34" y1="109.22" x2="53.34" y2="106.68" width="0.1524" layer="91"/>
+<pinref part="3.3VPI" gate="G$1" pin="10"/>
+<wire x1="53.34" y1="106.68" x2="48.26" y2="106.68" width="0.1524" layer="91"/>
+</segment>
+</net>
